Commit message: urdf update

File: src/fortnight/urdf/robot.urdf.xacro (robot description, xacro)
@@ -11,6 +11,11 @@
   <joint name="laser_base_joint" type="fixed">
 	  <!-- some parts are running on indigo, from jade , tehre is constant pi, use it instead on newer robots -->
+	  <!-- there are also no trigonometric functions in old versions, so we will compute it outside -->
 	  <xacro:property name="PI" value="3.14159265358979" />
-	  <origin rpy="${PI} 0 -${PI/4 + 0.01}" xyz="0.145 -0.15 0.095"/>
+	  <xacro:property name="radius" value=".206" />
+	  <xacro:property name="angle" value="${-PI/4 + 0.15}" />
+	  <xacro:property name="x" value="${ .80483545108964388920 * radius}" /> <!-- cos(angle) * distance -->
+	  <xacro:property name="y" value="${-.59349801740977150377 * radius}" /> <!-- sin(angle) * distance -->
+	  <origin rpy="${PI} 0 ${angle}" xyz="${x} ${y} 0.0908"/>
     	<parent link="base_link"/>
     	<child link="laser_mount_link"/>

Commit message: laser: final position

File: src/fortnight/urdf/robot.urdf.xacro (robot description, xacro)
@@ -13,9 +13,9 @@
 	  <!-- there are also no trigonometric functions in old versions, so we will compute it outside -->
 	  <xacro:property name="PI" value="3.14159265358979" />
-	  <xacro:property name="radius" value=".206" />
+	  <xacro:property name="radius" value=".201" />
 	  <xacro:property name="angle" value="${-PI/4 + 0.15}" />
 	  <xacro:property name="x" value="${ .80483545108964388920 * radius}" /> <!-- cos(angle) * distance -->
 	  <xacro:property name="y" value="${-.59349801740977150377 * radius}" /> <!-- sin(angle) * distance -->
-	  <origin rpy="${PI} 0 ${angle}" xyz="${x} ${y} 0.0908"/>
+	  <origin rpy="${PI} 0 ${angle}" xyz="${x} ${y} 0.127"/>
     	<parent link="base_link"/>
     	<child link="laser_mount_link"/>
